Commit message: GUI -v1

File: Scripts/mechanic_model_urdf/urdf/mechanic_model_urdf.urdf (robot description, URDF)
Before this commit: robot mechanic_model_exo6gdl, 7 links, 6 joints
Links:
- removed link inertial
- removed link link1
- removed link link2
- removed link link3
- removed link link4
- removed link link5
- removed link link6
- added link Link1, mass 0; collision mesh filename=package://mechanic_model_urdf/meshes/Link1.STL; visual mesh filename=package://mechanic_model_urdf/meshes/Link1.STL
- added link Link2, mass 0; collision mesh filename=package://mechanic_model_urdf/meshes/Link2.STL; visual mesh filename=package://mechanic_model_urdf/meshes/Link2.STL
- added link Link3, mass 0; collision mesh filename=package://mechanic_model_urdf/meshes/Link3.STL; visual mesh filename=package://mechanic_model_urdf/meshes/Link3.STL
- added link Link4, mass 0; collision mesh filename=package://mechanic_model_urdf/meshes/Link4.STL; visual mesh filename=package://mechanic_model_urdf/meshes/Link4.STL
- added link Link5, mass 0; collision mesh filename=package://mechanic_model_urdf/meshes/Link5.STL; visual mesh filename=package://mechanic_model_urdf/meshes/Link5.STL
- added link Link6, mass 0; collision mesh filename=package://mechanic_model_urdf/meshes/Link6.STL; visual mesh filename=package://mechanic_model_urdf/meshes/Link6.STL
- added link base_link, mass 0; collision mesh filename=package://mechanic_model_urdf/meshes/base_link.STL; visual mesh filename=package://mechanic_model_urdf/meshes/base_link.STL
Joints:
- joint q1: axis 0 -1 0 -> 0 1 0; child link1 -> Link1; parent inertial -> base_link
- joint q2: child link2 -> Link2; origin xyz=0.0323552493341545 0 0.105133904334066 rpy=0 0 0 -> xyz=0.032355 0 0.10513 rpy=0 0 0; parent link1 -> Link1
- joint q3: axis -0.831636482590333 0 0.555320412757156 -> -0.83164 0 0.55532; child link3 -> Link3; origin xyz=-0.0361375560878337 0 0.0250384839032992 rpy=0 0 0 -> xyz=-0.036138 0 0.025038 rpy=0 0 0; parent link2 -> Link2
- joint q4: axis 0 0 -1 -> 0 0 1; child link4 -> Link4; origin xyz=-0.0130095953517694 0 0.0228689244744532 rpy=0 0 0 -> xyz=-0.012178 0 0.021314 rpy=0 0 0; parent link3 -> Link3
- joint q5: child link5 -> Link5; origin xyz=-0.000179990761935058 0 0.042340751540877 rpy=0 0 0 -> xyz=-0.00017999 0 0.042341 rpy=0 0 0; parent link4 -> Link4
- joint q6: axis 0 -1 0 -> 0 1 0; child link6 -> Link6; origin xyz=0 0 0.00600000000000012 rpy=0 0 0 -> xyz=0 0 0.006 rpy=0 0 0; parent link5 -> Link5
